File: energy_harvester.kicad_sch (KiCad schematic)
At the start: 13 parts, among them IC1 LTC3108EGN-1-PBF, J1 Conn_01x02_Female, J2 Conn_01x02_Female, Q1 RUM002N02T2L

Commit message: Add traces, step files, corr in schematic
Connections:
- net at C1.1, J1.2 (Pin_2), L1.1: no longer C2.1, C3.1, L1.4
- new net: C2.1, C3.1, L1.4
Changed lines of the file:
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@@
   (junction (at 34.29 90.17) (diameter 0) (color 0 0 0 0))
   (junction (at 40.64 82.55) (diameter 0) (color 0 0 0 0))
-  (junction (at 54.61 73.66) (diameter 0) (color 0 0 0 0))
-  (junction (at 57.15 73.66) (diameter 0) (color 0 0 0 0))
   (junction (at 66.04 81.28) (diameter 0) (color 0 0 0 0))
   (junction (at 138.43 115.57) (diameter 0) (color 0 0 0 0))
@@
     (stroke (width 0) (type default) (color 0 0 0 0))
   )
-  (wire (pts (xy 54.61 73.66) (xy 57.15 73.66))
-    (stroke (width 0) (type default) (color 0 0 0 0))
-  )

Commit message: Change C value
Parts:
- C3: value 990p -> 1n
- C5: value 5u -> 4.7u
- IC1: value LTC3108EGN-1-PBF -> LTC3108EGN-1-TRPBF
Changed lines of the file:
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@@
     (in_bom yes) (on_board yes) (fields_autoplaced)
     (property "Reference" "C3" (id 0) (at 71.12 85.09 90))
-    (property "Value" "990p" (id 1) (at 71.12 87.63 90))
+    (property "Value" "1n" (id 1) (at 71.12 87.63 90))
     (property "Footprint" "Capacitor_SMD:C_0805_2012Metric_Pad1.18x1.45mm_HandSolder" (id 2) (at 71.12 91.44 0)
       (effects (font (size 1.27 1.27)) hide)
@@
       (effects (font (size 1.27 1.27)) (justify left))
     )
-    (property "Value" "5u" (id 1) (at 228.6 85.0899 0)
+    (property "Value" "4.7u" (id 1) (at 228.6 85.0899 0)
       (effects (font (size 1.27 1.27)) (justify left))
     )
@@
       (effects (font (size 1.524 1.524)))
     )
-    (property "Value" "LTC3108EGN-1-PBF" (id 1) (at 140.97 74.93 0)
+    (property "Value" "LTC3108EGN-1-TRPBF" (id 1) (at 140.97 74.93 0)
       (effects (font (size 1.524 1.524)))
     )
@@
     )
     (path "/86d69bc3-662d-4404-92e5-948b1cb0c889"
-      (reference "C3") (unit 1) (value "990p") (footprint "Capacitor_SMD:C_0805_2012Metric_Pad1.18x1.45mm_HandSolder")
+      (reference "C3") (unit 1) (value "1n") (footprint "Capacitor_SMD:C_0805_2012Metric_Pad1.18x1.45mm_HandSolder")
     )
     (path "/83a3f49d-acb8-484c-a6f3-f53aac9094cf"
@@
     )
     (path "/6acbf591-bff9-457a-95a0-80575e8c164f"
-      (reference "C5") (unit 1) (value "5u") (footprint "Capacitor_SMD:C_0805_2012Metric_Pad1.18x1.45mm_HandSolder")
+      (reference "C5") (unit 1) (value "4.7u") (footprint "Capacitor_SMD:C_0805_2012Metric_Pad1.18x1.45mm_HandSolder")
     )
     (path "/2f55abfa-582e-4300-a185-a37a87616fea"
-      (reference "IC1") (unit 1) (value "LTC3108EGN-1-PBF") (footprint "LTC3108:LTC3108EGN-1-PBF")
+      (reference "IC1") (unit 1) (value "LTC3108EGN-1-TRPBF") (footprint "LTC3108:LTC3108EGN-1-PBF")
     )
     (path "/1bfb43f6-53da-4112-8323-c6bee2d3244a"
