File: energy_harvester.kicad_pcb (KiCad board)
At the start: 2 copper layers, 60 x 25 mm, 13 parts, among them IC1 LTC3108EGN-1-PBF, J1 Conn_01x02_Female, J2 Conn_01x02_Female, Q1 RUM002N02T2L

Commit message: Pour Ground
Routing:
- net GND: track 154.3 -> 160.0 mm
- net Net-(J2-Pad2): track 25.3 -> 29.5 mm
- net /VAUX: track 18.7 -> 15.4 mm
- net /SW: track 10.0 -> 9.16 mm
Other:
- board text added: "Input: TEC1-12703 160mV Output: 3.3V"
- board text removed: "Input: TEC1-12703 80mV Output: 3V"
